File: kicad/esp32.kicad_sch (KiCad schematic)
At the start: 26 parts, among them J2 USB_C_Receptacle_USB2.0_14P, J3 Micro_SD_Card_Det2, U3 USBLC6-2SC6, U4 ESP32-S3-WROOM-1U-N16R8, U5 USBLC6-4SC6, U6 W25Q128JVS

Commit message: finished adding nets to mega2560 sheet
Connections:
- net IO38 renamed RTC_INT
Other:
- moved on the sheet: C4, D2, F2, J2, R5, R6, R7, R9, U3
