File: kicad/headers.kicad_sch (KiCad schematic)
At the start: 10 parts, among them J10 TC2030, J11 Conn_02x18_Odd_Even, J12 Conn_01x10, J13 Conn_01x08, J14 Conn_01x08, J15 Conn_02x06_Counter_Clockwise, J7 Conn_01x08, J8 Conn_01x08, J9 Conn_01x08, SW1 SW_SPST

Commit message: finished adding nets to mega2560 sheet
Connections:
- net Vin renamed VIN
Changed lines of the file:
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@@
+		)
+	)
+	(global_label "VIN"
+		(shape input)
+		(at 33.02 44.45 180)
+		(fields_autoplaced yes)
+		(effects
+			(font
+				(size 1.27 1.27)
+			)
+			(justify right)
+		)
+		(property "Intersheetrefs" "${INTERSHEET_REFS}"
+			(at 27.0109 44.45 0)
+			(hide yes)
+			(show_name no)
+			(do_not_autoplace no)
+			(effects
+				(font
+					(size 1.27 1.27)
+				)
+				(justify right)
+			)
 		)
 	)
@@
 		)
 	)
-	(hierarchical_label "Vin"
-		(shape input)
-		(at 33.02 44.45 180)
-		(effects
-			(font
-				(size 1.27 1.27)
-			)
-			(justify right)
-		)
-	)
