File: kicad/power.kicad_sch (KiCad schematic)
At the start: 19 parts, among them J4 2.1mm ID 5.5mm OD, Q1 DMP3013SFV, U10 TLV75733PDBV, U11 TLV75733PDBV, U9 TPS62163DSG

Commit message: finished adding nets to mega2560 sheet
Connections:
- net VIN: now reaches J4.1, Q1.5 (D)
Changed lines of the file:
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@@
 	(paper "A4")
 	(junction
+		(at 38.1 35.56)
+		(diameter 0)
+		(color 0 0 0 0)
+	)
+	(junction
 		(at 232.41 35.56)
 		(diameter 0)
@@
 	(wire
 		(pts
+			(xy 38.1 35.56) (xy 44.45 35.56)
+		)
+		(stroke
+			(width 0)
+			(type default)
+		)
+	)
+	(wire
+		(pts
 			(xy 130.81 39.37) (xy 130.81 35.56)
 		)
@@
 	(wire
 		(pts
-			(xy 33.02 35.56) (xy 44.45 35.56)
+			(xy 33.02 35.56) (xy 38.1 35.56)
 		)
 		(stroke
@@
 	(wire
 		(pts
+			(xy 38.1 34.29) (xy 38.1 35.56)
+		)
+		(stroke
+			(width 0)
+			(type default)
+		)
+	)
+	(wire
+		(pts
 			(xy 256.54 35.56) (xy 257.81 35.56)
 		)
@@
 		)
 	)
+	(global_label "VIN"
+		(shape input)
+		(at 38.1 34.29 90)
+		(fields_autoplaced yes)
+		(effects
+			(font
+				(size 1.27 1.27)
+			)
+			(justify left)
+		)
+		(property "Intersheetrefs" "${INTERSHEET_REFS}"
+			(at 38.1 28.2809 90)
+			(hide yes)
+			(show_name no)
+			(do_not_autoplace no)
+			(effects
+				(font
+					(size 1.27 1.27)
+				)
+				(justify left)
+			)
+		)
+	)
