File: kicad/peripherals.kicad_sch (KiCad schematic)
At the start: 7 parts, among them J5 Conn_01x04_MountingPin, J6 Conn_01x04_MountingPin, U15 DS3231M

Commit message: finished schematic and start pcb
Parts:
- added C33, C34, C35, C38, C39, C40, C41, C42: 0.1uF, Capacitor_SMD:C_0603_1608Metric, symbol Device:C_Small
- added D10: WHITE, LED_SMD:LED_Avago_PLCC4_3.2x2.8mm_CW, symbol Device:LED
- added D11, D12: RED, LED_SMD:LED_Avago_PLCC4_3.2x2.8mm_CW, symbol Device:LED
- added D13, D17, D19, D20, D3, D4, D5, D9: WS2812B-2020, LED_SMD:LED_WS2812B-2020_PLCC4_2.0x2.0mm, symbol LED:WS2812B-2020
- added D14, D15, D16: GREEN, LED_SMD:LED_Avago_PLCC4_3.2x2.8mm_CW, symbol Device:LED
- added D18: YELLOW, LED_SMD:LED_Avago_PLCC4_3.2x2.8mm_CW, symbol Device:LED
- added D6: BLUE, LED_SMD:LED_Avago_PLCC4_3.2x2.8mm_CW, symbol Device:LED
- added D7: PURPLE, LED_SMD:LED_Avago_PLCC4_3.2x2.8mm_CW, symbol Device:LED
- added D8: ORANGE, LED_SMD:LED_Avago_PLCC4_3.2x2.8mm_CW, symbol Device:LED
- added R24, R25, R26, R27, R28, R29, R30, R31: 1k, Resistor_SMD:R_0603_1608Metric, symbol Device:R_Small_US
- added R32, R33: 2.2k, Resistor_SMD:R_0603_1608Metric, symbol Device:R_Small_US
- C36: renamed from C33; footprint (none) -> Capacitor_SMD:C_0603_1608Metric
- C37: renamed from C34; footprint (none) -> Capacitor_SMD:C_0603_1608Metric
- R23: renamed from R21; footprint (none) -> Resistor_SMD:R_0603_1608Metric
Connections:
- net +3.3VP: now also R30.1
- net +5V: now also C33.1, C34.1, C35.1, C38.1, C39.1, C40.1, C41.1, C42.1, D13.4 (VDD), D17.4 (VDD), D19.4 (VDD), D20.4 (VDD), D3.4 (VDD), D4.4 (VDD), D5.4 (VDD), D9.4 (VDD), R32.1
- net GND: now also C33.2, C34.2, C35.2, C38.2, C39.2, C40.2, C41.2, C42.2, D10.1 (K), D11.1 (K), D12.1 (K), D13.2 (VSS), D14.1 (K), D15.1 (K), D16.1 (K), D17.2 (VSS), D18.1 (K), D19.2 (VSS), D20.2 (VSS), D3.2 (VSS), D4.2 (VSS), D5.2 (VSS), D6.1 (K), D7.1 (K), D8.1 (K), D9.2 (VSS)
- net 5V_I2C_SCL renamed AVR_SCL
- net 5V_I2C_SDA renamed AVR_SDA
- new net: D18.2 (A), R33.2
- new net: D3.1 (DOUT), D4.3 (DIN)
- new net: D13.1 (DOUT), D17.3 (DIN)
- new net: D13.3 (DIN), D9.1 (DOUT)
- new net: D8.2 (A), R26.2
- new net: D12.2 (A), R29.2
- new net: D5.1 (DOUT), D9.3 (DIN)
- new net: D4.1 (DOUT), D5.3 (DIN)
- new net: D11.2 (A), R28.2
- new net: D16.2 (A), R32.2
- new net: D14.2 (A), R30.2
- new net: D6.2 (A), R24.2
- new net: D19.1 (DOUT), D20.3 (DIN)
- new net: D10.2 (A), R27.2
- new net: D17.1 (DOUT), D19.3 (DIN)
- new net: D15.2 (A), R31.2
- new net: D7.2 (A), R25.2
- new net +3.3V: R31.1
- new net AVR_USER_LED: R33.1
- new net ESP_USER_LED: R24.1
- new net LED_CBUS0: R29.1
- new net LED_CBUS1: R28.1
- new net LED_CBUS2: R27.1
- new net LED_CBUS3: R26.1
- new net LED_NPX: D3.3 (DIN)
- new net LED_uSD: R25.1
- no-connect marks 1 -> 2
Other:
- note removed: "LEDs here too!"
