File: kicad/_restore_backup_2026-08-04T15-06-31-186/Mega2560plus.kicad_sch (KiCad schematic)
At the start: 6 parts

Commit message: finished schematic and start pcb
Other:
- sheet ESP32 ports: added IO39; removed ESP32_NPX
- sheet Headers ports: added IO39; removed ESP_BOOT0, ESP_RESET
- sheet Peripherals ports: added none; removed AVR_USER_LED, ESP_USER_LED, LED_CBUS0, LED_CBUS1, LED_CBUS2, LED_CBUS3, LED_NPX, LED_uSD
