File: kicad/_restore_backup_2026-08-04T15-06-31-186/power.kicad_sch (KiCad schematic)
At the start: 19 parts, among them J4 2.1mm ID 5.5mm OD PJ-102AH, Q1 DMP3013SFV, U10 TLV75733PDBV, U11 TLV75733PDBV, U9 TPS62163DSG

Commit message: finished schematic and start pcb
Parts:
- C17, C18, C19, C20, C21, C22, C23, C24, C25, C26, C27: footprint Capacitor_SMD:C_0603_1608Metric -> (none)
- J4: value 2.1mm ID 5.5mm OD PJ-102AH -> 2.1mm ID 5.5mm OD; footprint Connector_BarrelJack:BarrelJack_CUI_PJ-102AH_Horizontal -> PJ-102AH
- L1: value 2.2uH Coilcraft XAL5030-222MEC -> 2.2uH; footprint Inductor_SMD:L_Coilcraft_XAL5030-XXX -> (none)
- R20, R21: footprint Resistor_SMD:R_0603_1608Metric -> (none)
Changed lines of the file:
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@@
 			)
 		)
-		(property "Footprint" "Capacitor_SMD:C_0603_1608Metric"
+		(property "Footprint" ""
 			(at 267.97 39.37 0)
 			(hide yes)
@@
 			)
 		)
-		(property "Value" "2.1mm ID 5.5mm OD PJ-102AH"
+		(property "Value" "2.1mm ID 5.5mm OD"
 			(at 25.4 31.75 0)
 			(show_name no)
@@
 			)
 		)
-		(property "Footprint" "Connector_BarrelJack:BarrelJack_CUI_PJ-102AH_Horizontal"
+		(property "Footprint" "PJ-102AH"
 			(at 26.67 39.116 0)
 			(hide yes)
@@
 			)
 		)
-		(property "Footprint" "Capacitor_SMD:C_0603_1608Metric"
+		(property "Footprint" ""
 			(at 222.25 39.37 0)
 			(hide yes)
@@
 			)
 		)
-		(property "Footprint" "Capacitor_SMD:C_0603_1608Metric"
+		(property "Footprint" ""
 			(at 267.97 67.31 0)
 			(hide yes)
@@
 			)
 		)
-		(property "Footprint" "Capacitor_SMD:C_0603_1608Metric"
+		(property "Footprint" ""
 			(at 86.36 39.37 0)
 			(hide yes)
@@
 			)
 		)
-		(property "Footprint" "Capacitor_SMD:C_0603_1608Metric"
+		(property "Footprint" ""
 			(at 232.41 39.37 0)
 			(hide yes)
@@
 			)
 		)
-		(property "Footprint" "Resistor_SMD:R_0603_1608Metric"
+		(property "Footprint" ""
 			(at 90.17 50.8 0)
 			(hide yes)
@@
 			)
 		)
-		(property "Footprint" "Capacitor_SMD:C_0603_1608Metric"
+		(property "Footprint" ""
 			(at 257.81 39.37 0)
 			(hide yes)
@@
 			)
 		)
-		(property "Footprint" "Capacitor_SMD:C_0603_1608Metric"
+		(property "Footprint" ""
 			(at 257.81 67.31 0)
 			(hide yes)
@@
 			)
 		)
-		(property "Footprint" "Capacitor_SMD:C_0603_1608Metric"
+		(property "Footprint" ""
 			(at 76.2 39.37 0)
 			(hide yes)
@@
 			)
 		)
-		(property "Footprint" "Capacitor_SMD:C_0603_1608Metric"
+		(property "Footprint" ""
 			(at 232.41 67.31 0)
 			(hide yes)
@@
 			)
 		)
-		(property "Footprint" "Capacitor_SMD:C_0603_1608Metric"
+		(property "Footprint" ""
 			(at 222.25 67.31 0)
 			(hide yes)
@@
 			)
 		)
-		(property "Footprint" "Resistor_SMD:R_0603_1608Metric"
+		(property "Footprint" ""
 			(at 49.53 46.99 0)
 			(hide yes)
@@
 			)
 		)
-		(property "Value" "2.2uH Coilcraft XAL5030-222MEC"
+		(property "Value" "2.2uH"
 			(at 121.92 33.02 90)
 			(show_name no)
@@
 			)
 		)
-		(property "Footprint" "Inductor_SMD:L_Coilcraft_XAL5030-XXX"
+		(property "Footprint" ""
 			(at 121.92 35.56 0)
 			(hide yes)
@@
 			)
 		)
-		(property "Footprint" "Capacitor_SMD:C_0603_1608Metric"
+		(property "Footprint" ""
 			(at 130.81 41.91 0)
 			(hide yes)
