File: kicad/_restore_backup_2026-08-04T18-34-35-782/peripherals.kicad_sch (KiCad schematic)
At the start: 43 parts, among them J5 Conn_01x04_MountingPin, J6 Conn_01x04_MountingPin, U15 DS3231M

Commit message: finish pcb
Parts:
- BT1: footprint Battery:BatteryHolder_LINX_BAT-HLD-012-SMT -> Battery:BatteryHolder_Keystone_1060_1x2032
- C36, C37: footprint Capacitor_SMD:C_0402_1005Metric -> Capacitor_SMD:C_0603_1608Metric
- D10, D11, D12, D14, D15, D16, D18, D6, D7, D8: footprint LED_SMD:LED_0402_1005Metric -> LED_SMD:LED_Avago_PLCC4_3.2x2.8mm_CW
- J5, J6: footprint Connector_JST:JST_SH_BM04B-SRSS-TB_1x04-1MP_P1.00mm_Vertical -> Connector_JST:JST_SH_SM04B-SRSS-TB_1x04-1MP_P1.00mm_Horizontal
- R24: renamed from R22; footprint Resistor_SMD:R_0402_1005Metric -> Resistor_SMD:R_0603_1608Metric
- R25: renamed from R23; footprint Resistor_SMD:R_0402_1005Metric -> Resistor_SMD:R_0603_1608Metric
- R26: renamed from R24; footprint Resistor_SMD:R_0402_1005Metric -> Resistor_SMD:R_0603_1608Metric
- R27: renamed from R25; footprint Resistor_SMD:R_0402_1005Metric -> Resistor_SMD:R_0603_1608Metric
- R28: renamed from R26; footprint Resistor_SMD:R_0402_1005Metric -> Resistor_SMD:R_0603_1608Metric
- R29: renamed from R27; footprint Resistor_SMD:R_0402_1005Metric -> Resistor_SMD:R_0603_1608Metric
- R30: renamed from R28; footprint Resistor_SMD:R_0402_1005Metric -> Resistor_SMD:R_0603_1608Metric
- R31: renamed from R29; footprint Resistor_SMD:R_0402_1005Metric -> Resistor_SMD:R_0603_1608Metric
- R32: renamed from R30; footprint Resistor_SMD:R_0402_1005Metric -> Resistor_SMD:R_0603_1608Metric
- R33: renamed from R31; footprint Resistor_SMD:R_0402_1005Metric -> Resistor_SMD:R_0603_1608Metric
- renumbered R21 to R23
